File: radio20-synth/A2.kicad_sch (KiCad schematic)
At the start: 143 parts, among them Q1 КТ315Г, Q2 КТ315Г, Q3 КТ361Г, Q4 КП307Г, Q5 КТ372В, U1 К155ТМ2, U2 К155ЛА3, U3 К500ЛМ102

Commit message: Fix typo in A2 sheet title by changing it
Parts:
- C15: value (none) -> 100uF 10V
- C19, C20, C21, C43, J5, R21: value (none) -> ~
- D1: value (none) -> КД503А; footprint (none) -> Diode_THT:D_DO-35_SOD27_P7.62mm_Horizontal
- D10, D9: value (none) -> КД103А
- D11, D12, D13, D14, D15, D16, D17, D18: value (none) -> КА517А
- J1, J2, J3, J4: value (none) -> Conn_Coaxial
- L3: value (none) -> 200uH
- R10001, R10002: value (none) -> 0
- R17: value (none) -> 75
- R18: value (none) -> 1K
- R19, R20: value (none) -> 330
- R29, R30, R31, R32, R33, R34, R35: value (none) -> 33K
- R36: value (none) -> 33K; footprint (none) -> 33K
Connections:
- new net: D18.1 (K), W8., W9.
- new net: D12.1 (K), W1., W3.
- new net: D16.1 (K), W6., W7.
Other:
- title: А2: Имулсно-фазов детектор, ФНЧ. ГУН -> Синтезатор на честота, Радио/1990/1,2,3
