File: radio20-synth/radio20-synth.kicad_sch (KiCad schematic)
At the start: 43 parts, among them Q1 КТ315Г, Q2 КТ315Г, Q3 КТ361Г, U1 К155ТМ2, U2 К155ЛА3

Commit message: A2 module almost done; A2.pdf plot rendering
Parts:
- removed C1, C?: 300uF 25V, symbol Device:C_Polarized
- removed C10, C2, C3, C52: 150nF, symbol Device:C
- removed C11: 68pF, symbol Device:C
- removed C4, C8: 15nF, symbol Device:C
- removed C5: 33uF 24V, symbol Device:C_Polarized
- removed C51: 300uF 15V, symbol Device:C_Polarized
- removed C6: 3.3uF 24V, symbol Device:C_Polarized
- removed C7: 1uF 30V, symbol Device:C_Polarized
- removed D1: КД503А, Diode_THT:D_DO-35_SOD27_P7.62mm_Horizontal, symbol Diode:BAW76
- removed D2: КС213Б, symbol Device:D_TVS
- removed D3, D4, D5, D6, D7, D8: КВ109Б, symbol Device:D_Capacitance
- removed L1, L4: 250uH, symbol Device:L_Ferrite
- removed Q1: КТ315Г, Package_TO_SOT_THT:TO-92, symbol Transistor_BJT:BC413C
- removed Q2: КТ315Г, Package_TO_SOT_THT:TO-92_Inline, symbol Transistor_BJT:BC413C
- removed Q3: КТ361Г, Package_TO_SOT_THT:TO-92_Inline, symbol Transistor_BJT:BC559
- removed Q4: (no value), symbol радио20:КП307Г
- removed R1, R2, R5, R6: 680, symbol Device:R_Small
- removed R10: 51K, symbol Device:R_Small
- removed R10000, R10001: 0, symbol Device:R_Small
- removed R11, R12: 100K, symbol Device:R_Small
- removed R3: 9.1K, symbol Device:R_Small
- removed R4: 3K, symbol Device:R_Small
- removed R7: 910, symbol Device:R_Small
- removed R8: 2.4K, symbol Device:R_Small
- removed R9: 2K, symbol Device:R_Small
- removed U1: К155ТМ2, symbol радио20:К155ТМ2
- removed U2: К155ЛА3, symbol радио20:К155ЛА3
Connections:
- no-connect marks 2 -> 0
Other:
- added sheet A1 (A1.kicad_sch)
- added sheet A2 (A2.kicad_sch)
- added sheet A3 (A3.kicad_sch)
- note removed: "А2: Импулсно-фазов детектор, ФНЧ, ГУН"
- title: (none) -> А2: Имулсно-фазов детектор, ФНЧ. ГУН

Commit message: Fix typo in A2 sheet title by changing it
Other:
- title: А2: Имулсно-фазов детектор, ФНЧ. ГУН -> Синтезатор на честота, Радио/1990/1,2,3
Changed lines of the file:
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@@
   (paper "A4")
   (title_block
-    (title "А2: Имулсно-фазов детектор, ФНЧ. ГУН")
+    (title "Синтезатор на честота, Радио/1990/1,2,3")
   )
   (sheet (at 100.965 111.76) (size 39.37 22.86) (fields_autoplaced)
